File: STM32F4_REV2.sch (KiCad schematic (older format))
At the start: 50 parts, among them J1 Screw_Terminal_01x02, J2 SWD, J3 Conn_01x04, J4 Conn_01x04, J5 USB_B_Micro, Q1 AO3401A, SW1 SW_SPDT, U1 MP2359DJ-LF-Z, U2 STM32F405RGT6, U3 USBLC6-2SC6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

Commit message: compile
Parts:
- J5: symbol Connector:USB_B_Micro -> STM32F4_REV2-rescue:USB_B_Micro-Connector
- U1: symbol SchmillipKiCADLibrary:MP2359DJ-LF-Z -> STM32F4_REV2-rescue:MP2359DJ-LF-Z-SchmillipKiCADLibrary
Changed lines of the file:
@@
 	1000 6750 1000 6650
 $Comp
-L SchmillipKiCADLibrary:MP2359DJ-LF-Z U1
+L STM32F4_REV2-rescue:MP2359DJ-LF-Z-SchmillipKiCADLibrary U1
 U 1 1 5F7EC586
 P 5825 1250
@@
 USART3_RX
 $Comp
-L Connector:USB_B_Micro J5
+L STM32F4_REV2-rescue:USB_B_Micro-Connector J5
 U 1 1 5F973FD8
 P 6775 5600
